File: TPS_Calibration_Board.kicad_pcb (KiCad board)
At the start: 4 copper layers, 57 x 47.8 mm, 44 parts, among them J1 VEHICLE SIDE, J2 TPS SIDE, J3 PROG, P1 HID, Q1 AO3407, SW1 RESET, U1 25LC1024, U2 STM32G431K6Tx, U3 FT230XQ, U4 TPS5430DDA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

Commit message: Minor changes
Parts:
- moved SW1 1.25 mm to (150.8, 90.0), turned to -90 degrees
Routing:
- net GND: track 100.3 -> 102.0 mm
- net NRST: track 47.0 -> 46.2 mm
Other:
- board text added: "5V SIG GND"
- board text added: "NRST SWDIO GND SWCLK 3.3V"
Changed lines of the file:
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@@
 		)
 		(property "Value" "TPS SIDE"
-			(at 0 7.41 360)
-			(layer "F.Fab")
+			(at 3 2.275 -90)
+			(unlocked yes)
+			(layer "F.SilkS")
 			(effects
 				(font
-					(size 1 1)
-					(thickness 0.15)
+					(size 0.5 0.5)
+					(thickness 0.125)
 				)
 			)
@@
 		)
 		(property "Value" "VEHICLE SIDE"
-			(at 0 7.41 360)
-			(layer "F.Fab")
+			(at 3 2.83 -90)
+			(unlocked yes)
+			(layer "F.SilkS")
 			(effects
 				(font
-					(size 1 1)
-					(thickness 0.15)
+					(size 0.5 0.5)
+					(thickness 0.125)
 				)
 			)
@@
 	(footprint "Button_Switch_SMD:SW_SPST_B3S-1000"
 		(layer "F.Cu")
-		(at 149.5 90 180)
+		(at 150.75 90.025 -90)
 		(descr "Surface Mount Tactile Switch for High-Density Packaging")
 		(tags "Tactile Switch")
 		(property "Reference" "SW1"
-			(at 0 -4.5 360)
+			(at 0 -4.5 90)
 			(layer "F.SilkS")
 			(effects
@@
 		)
 		(property "Value" "RESET"
-			(at 0 4.5 360)
-			(layer "F.Fab")
+			(at 0.475 -5.75 90)
+			(unlocked yes)
+			(layer "F.SilkS")
+			(hide yes)
 			(effects
 				(font
-					(size 1 1)
-					(thickness 0.15)
+					(size 0.5 0.5)
+					(thickness 0.125)
 				)
 			)
 		)
 		(property "Footprint" "Button_Switch_SMD:SW_SPST_B3S-1000"
-			(at 0 0 180)
+			(at 0 0 -90)
 			(unlocked yes)
 			(layer "F.Fab")
@@
 		)
 		(property "Datasheet" ""
-			(at 0 0 180)
+			(at 0 0 -90)
 			(unlocked yes)
 			(layer "F.Fab")
@@
 		)
 		(property "Description" "Push button switch, generic, two pins"
-			(at 0 0 180)
+			(at 0 0 -90)
 			(unlocked yes)
 			(layer "F.Fab")
@@
 		(attr smd)
 		(fp_line
-			(start 3.15 3.45)
-			(end -3.15 3.45)
+			(start -3.15 3.45)
+			(end -3.15 3.2)
 			(stroke
 				(width 0.12)
@@
 		)
 		(fp_line
-			(start 3.15 3.2)
-			(end 3.15 3.45)
+			(start 3.15 3.45)
+			(end -3.15 3.45)
 			(stroke
 				(width 0.12)
@@
 		)
 		(fp_line
-			(start 3.15 -1.3)
-			(end 3.15 1.3)
+			(start 3.15 3.2)
+			(end 3.15 3.45)
 			(stroke
 				(width 0.12)
@@
 		)
 		(fp_line
-			(start 3.15 -3.45)
-			(end 3.15 -3.2)
+			(start -3.15 1.3)
+			(end -3.15 -1.3)
 			(stroke
 				(width 0.12)
@@
 		)
 		(fp_line
-			(start -3.15 3.45)
-			(end -3.15 3.2)
+			(start 3.15 -1.3)
+			(end 3.15 1.3)
 			(stroke
 				(width 0.12)
@@
 		)
 		(fp_line
-			(start -3.15 1.3)
-			(end -3.15 -1.3)
+			(start -3.15 -3.2)
+			(end -3.15 -3.45)
 			(stroke
 				(width 0.12)
@@
 		)
 		(fp_line
-			(start -3.15 -3.2)
-			(end -3.15 -3.45)
+			(start -3.15 -3.45)
+			(end 3.15 -3.45)
 			(stroke
 				(width 0.12)
@@
 		)
 		(fp_line
-			(start -3.15 -3.45)
-			(end 3.15 -3.45)
+			(start 3.15 -3.45)
+			(end 3.15 -3.2)
 			(stroke
 				(width 0.12)
@@
 		)
 		(fp_line
-			(start 5 3.7)
-			(end 5 -3.7)
+			(start -5 3.7)
+			(end 5 3.7)
 			(stroke
 				(width 0.05)
@@
 		)
 		(fp_line
-			(start 5 -3.7)
-			(end -5 -3.7)
+			(start 5 3.7)
+			(end 5 -3.7)
 			(stroke
 				(width 0.05)
@@
 		)
 		(fp_line
-			(start -5 3.7)
-			(end 5 3.7)
+			(start -5 -3.7)
+			(end -5 3.7)
 			(stroke
 				(width 0.05)
@@
 		)
 		(fp_line
-			(start -5 -3.7)
-			(end -5 3.7)
+			(start 5 -3.7)
+			(end -5 -3.7)
 			(stroke
 				(width 0.05)
@@
 		)
 		(fp_line
-			(start 3 3.3)
-			(end -3 3.3)
+			(start -3 3.3)
+			(end -3 -3.3)
 			(stroke
 				(width 0.1)
@@
 		)
 		(fp_line
-			(start 3 -3.3)
-			(end 3 3.3)
+			(start 3 3.3)
+			(end -3 3.3)
 			(stroke
 				(width 0.1)
@@
 		)
 		(fp_line
-			(start -3 3.3)
-			(end -3 -3.3)
+			(start -3 -3.3)
+			(end 3 -3.3)
 			(stroke
 				(width 0.1)
@@
 		)
 		(fp_line
-			(start -3 -3.3)
-			(end 3 -3.3)
+			(start 3 -3.3)
+			(end 3 3.3)
 			(stroke
 				(width 0.1)
@@
 		)
 		(fp_text user "${REFERENCE}"
-			(at 0 -4.5 360)
+			(at 0 -4.5 90)
 			(layer "F.Fab")
 			(effects
@@
 		)
 		(pad "1" smd rect
-			(at -3.975 -2.25 180)
+			(at -3.975 -2.25 270)
 			(size 1.55 1.3)
 			(layers "F.Cu" "F.Paste" "F.Mask")
@@
 		)
 		(pad "1" smd rect
-			(at 3.975 -2.25 180)
+			(at 3.975 -2.25 270)
 			(size 1.55 1.3)
 			(layers "F.Cu" "F.Paste" "F.Mask")
@@
 		)
 		(pad "2" smd rect
-			(at -3.975 2.25 180)
+			(at -3.975 2.25 270)
 			(size 1.55 1.3)
 			(layers "F.Cu" "F.Paste" "F.Mask")
@@
 		)
 		(pad "2" smd rect
-			(at 3.975 2.25 180)
+			(at 3.975 2.25 270)
 			(size 1.55 1.3)
 			(layers "F.Cu" "F.Paste" "F.Mask")
@@
 		)
 	)
+	(gr_text "5V    SIG    GND"
+		(at 143.5 118.5 270)
+		(layer "F.SilkS")
+		(effects
+			(font
+				(size 0.5 0.5)
+				(thickness 0.125)
+			)
+		)
+	)
 	(gr_text "P/N: 0001-R00.\n"
 		(at 141.5 94.75 270)
@@
 		)
 	)
+	(gr_text "5V    SIG    GND"
+		(at 143.5 90 270)
+		(layer "F.SilkS")
+		(effects
+			(font
+				(size 0.5 0.5)
+				(thickness 0.125)
+			)
+		)
+	)
+	(gr_text "NRST SWDIO GND SWCLK  3.3V\n"
+		(at 168.5 86.5 180)
+		(layer "F.SilkS")
+		(effects
+			(font
+				(size 0.5 0.5)
+				(thickness 0.125)
+				(bold yes)
+			)
+			(justify left bottom)
+		)
+	)
 	(segment
 		(start 187.25 92)
@@
 	)
 	(segment
-		(start 153.475 87.75)
-		(end 155 89.275)
-		(width 0.2)
-		(layer "F.Cu")
-		(net 1)
-	)
-	(segment
 		(start 188.07 93.32)
 		(end 187 92.25)
@@
 	)
 	(segment
-		(start 155 89.275)
-		(end 155 89.5)
-		(width 0.2)
-		(layer "F.Cu")
-		(net 1)
-	)
-	(segment
 		(start 176 110.85)
 		(end 172.9 110.85)
@@
 	)
 	(segment
+		(start 148.5 86.05)
+		(end 148.5 94)
+		(width 0.25)
+		(layer "F.Cu")
+		(net 1)
+	)
+	(segment
 		(start 162.48 84.75)
 		(end 162.5 84.77)
@@
 	)
 	(segment
-		(start 188.7 92)
-		(end 189.9 92)
-		(width 0.2)
+		(start 151.5 96.5)
+		(end 151 96.5)
+		(width 0.25)
 		(layer "F.Cu")
 		(net 1)
 	)
 	(segment
-		(start 145.525 87.75)
-		(end 153.475 87.75)
+		(start 188.7 92)
+		(end 189.9 92)
 		(width 0.2)
 		(layer "F.Cu")
@@
 	)
 	(segment
+		(start 151 96.5)
+		(end 148.5 94)
+		(width 0.25)
+		(layer "F.Cu")
+		(net 1)
+	)
+	(segment
 		(start 193.05 97.25)
 		(end 193.05 94.74)
@@
 	)
 	(via
-		(at 160.5 103.75)
+		(at 151.5 96.5)
 		(size 0.6)
 		(drill 0.3)
@@
 	)
 	(via
-		(at 186.5 86.25)
+		(at 160.5 103.75)
 		(size 0.6)
 		(drill 0.3)
@@
 	)
 	(via
-		(at 167.5 91.25)
+		(at 186.5 86.25)
 		(size 0.6)
 		(drill 0.3)
@@
 	)
 	(via
-		(at 155 89.5)
+		(at 167.5 91.25)
 		(size 0.6)
 		(drill 0.3)
@@
 	)
 	(segment
+		(start 153 95)
+		(end 153 94)
+		(width 0.2)
+		(layer "F.Cu")
+		(net 3)
+	)
+	(segment
 		(start 154.975 100.225)
 		(end 155 100.25)
@@
 	)
 	(segment
-		(start 153.475 93.475)
-		(end 155.592157 95.592157)
+		(start 153 94)
+		(end 153 86.05)
 		(width 0.2)
 		(layer "F.Cu")
@@
 	)
 	(segment
-		(start 159.5 102.25)
-		(end 159.5 102.184314)
+		(start 154.975 96.209314)
+		(end 154.209314 96.209314)
 		(width 0.2)
 		(layer "F.Cu")
@@
 	)
 	(segment
-		(start 153.475 92.25)
-		(end 145.525 92.25)
+		(start 154.209314 96.209314)
+		(end 153 95)
 		(width 0.2)
 		(layer "F.Cu")
@@
 	)
 	(segment
-		(start 154.975 96.209314)
-		(end 154.975 97.5)
+		(start 159.5 102.25)
+		(end 159.5 102.184314)
 		(width 0.2)
 		(layer "F.Cu")
@@
 	)
 	(segment
-		(start 153.475 92.25)
-		(end 153.475 93.475)
+		(start 154.975 96.209314)
+		(end 154.975 97.5)
 		(width 0.2)
 		(layer "F.Cu")
